File: smart meter.kicad_sch (KiCad schematic)
At the start: 15 parts, among them J1 Energy_Meter_Conn, J2 Control_Terminal, J4 PV, J5 AC_Input, J6 DC_out, J7 Loads1, J8 Loads2

Commit message: Routing Power ctr
Parts:
- added H1, H2, H3, H4: MountingHole, MountingHole:MountingHole_3mm, symbol Mechanical:MountingHole
