File: Control board/Control_board/Control_board.kicad_sch (KiCad schematic)
At the start: 72 parts, among them J1 KEYPAD, J2 UART_conn, J3 Power_IN, J4 SPI_conn, J5 Triac Control, SW1 RESET, SW2 Button1, SW3 Button2, U1 AT45DB321E-SHF-T, U10 SP3485EN, U11 Debug, U12 PCA9554AD_118, U13 LM317DCY, U2 LM2576HVS-5, U3 LoRa, U4 Wifi, U6 STM32F103C8Tx, U7 RTC_DS3234, U8 DS3232SN-T&R, U9 OLED, Y1 8MHZ

Commit message: last edit
Parts:
- added C11: 100nF, Capacitor_SMD:C_0201_0603Metric, symbol Device:C
- added C12: 100uF, Capacitor_SMD:CP_Elec_6.3x7.7, symbol Device:C_Polarized_US
- added D10: 1N4007, Diode_SMD:D_SMA, symbol Diode:1N4007
- added D11: LED, symbol Device:LED
- added D12, D13: LED, LED_SMD:LED_0805_2012Metric, symbol Device:LED
- added J7: UART_wifi, smart_meter:RC4, symbol Connector:Screw_Terminal_01x04
- added J8: USB_B, symbol Connector:USB_B
- added JP3, JP?: Jumper_2_Open, symbol Jumper:Jumper_2_Open
- added R32, R40: 4.7K, symbol Device:R
- added R33, R34: 20, Resistor_SMD:R_1206_3216Metric, symbol Device:R
- added R35: 4.7K, Resistor_SMD:R_1206_3216Metric, symbol Device:R
- added R36, R37, R39: 470, Resistor_SMD:R_1206_3216Metric, symbol Device:R
- added R38: 0, Resistor_SMD:R_1206_3216Metric, symbol Device:R
- added R41, R42, R43, R44: 12K, Resistor_SMD:R_1206_3216Metric, symbol Device:R
- added R45: 10K, Resistor_SMD:R_1206_3216Metric, symbol Device:R
- added R46, R47: 150, Resistor_SMD:R_1206_3216Metric, symbol Device:R
- added SW4: KEY_flash, Button_Switch_SMD:SW_Tactile_SPST_NO_Straight_CK_PTS636Sx25SMTRLFS, symbol Switch:SW_Push
- added SW5: wifi_reset, Button_Switch_SMD:SW_Tactile_SPST_NO_Straight_CK_PTS636Sx25SMTRLFS, symbol Switch:SW_Push
- added SW6: Button1, Button_Switch_SMD:SW_Tactile_SPST_NO_Straight_CK_PTS636Sx25SMTRLFS, symbol Switch:SW_Push
- added U5: Olimex_MOD-WIFI-ESP8266-DEV, Module:Olimex_MOD-WIFI-ESP8266-DEV, symbol MCU_Module:Olimex_MOD-WIFI-ESP8266-DEV
- R1, R2, R3: value 10K -> 103
- R5: value 10K -> 12K
Connections:
- net 3.3V: now also U11.1 (Pin_1), C12.1, J7.2 (Pin_2), R32.2, R37.2, R40.1, R41.2, R42.2, R43.2, R45.2, U5.1 (3.3V); no longer J2.1 (Pin_1), U11.2 (Pin_2), U4.CH_PC, U4.GPIO0
- net 5V: now also J2.2 (Pin_2), D10.2 (A), J8.1 (VBUS), R35.1; no longer C5.1, U13.3 (INPUT)
- net Button1: now also U5.22 (GPIO4); no longer U6.2 (PC13)
- net Button2: now also U5.11 (GPIO5); no longer U6.3 (PC14)
- net DIO0: now also U6.2 (PC13); no longer U6.32 (PA11)
- net GND: now also J2.1 (Pin_1), U11.2 (Pin_2), C11.2, C12.2, D12.1 (K), D13.1 (K), J7.1 (Pin_1), J8.4 (GND), J8.5 (Shield), R44.2, SW4.2, SW5.2, SW6.2, U5.2 (GND); no longer J2.2 (Pin_2), U11.1 (Pin_1), U4.GPIO15
- net RST_LoRa: now also U6.3 (PC14); no longer U6.33 (PA12)
- net RST_WIFI: now also C11.1, R39.2, R43.1, U5.13 (RSTB); no longer R5.1
- net RX2: now also J2.3 (Pin_3); no longer J2.4 (Pin_4)
- net RX3: now also U4.TX, J7.3 (Pin_3), JP3.2 (B), U5.3 (GPIO1); no longer U4.RX, U6.22 (PB11)
- net SWCLK: now also U11.3 (Pin_3); no longer U11.4 (Pin_4)
- net SWDIO: now also U11.4 (Pin_4); no longer U11.3 (Pin_3)
- net TX2: now also J2.4 (Pin_4); no longer J2.3 (Pin_3)
- net TX3: now also U4.RX, J7.4 (Pin_4), JP?.2 (B), U5.4 (GPIO3); no longer U4.TX, U6.21 (PB10)
- net at U8.3 (32KHZ): now also R40.2
- net at U8.5 (*INT/SQW): now also R32.1
- net GPIO2: now reaches U4.GPIO2
- net GPIO2: now also R41.1, U5.20 (GPIO-2)
- net RST_flash: no longer names the net of R2.1, U1.3 (~{RESET})
- net RST_flash: no longer U6.10 (PA0)
- new net: C5.1, D10.1 (K), U13.3 (INPUT)
- new net: D11.2 (A), R37.1
- new net: D13.2 (A), R47.2
- new net: R38.1, R39.1, SW5.1
- new net: J8.2 (D-), R34.2
- new net: J8.3 (D+), R33.2
- new net: R36.1, SW4.1
- new net: D12.2 (A), R46.2
- new net Button3: R45.1, SW6.1, U5.16 (GPIO12)
- new net EN: R42.1, U4.CH_PC, U5.14 (CHIP_E)
- new net GPIO0: R36.2, R5.1, U4.GPIO0, U5.21 (GPIO-0)
- new net GPIO15: R44.1, U4.GPIO15, U5.19 (GPIO15)
- new net GPIO16: D11.1 (K), R38.2
- new net LED 1: R46.1, U5.18 (GPIO13)
- new net LED 2: R47.1, U5.17 (GPIO14)
- new net RX3_stm: JP3.1 (A), U6.22 (PB11)
- new net TX3_stm: JP?.1 (A), U6.21 (PB10)
- new net USB_DM: R34.1, U6.32 (PA11)
- new net USB_DP: R33.1, R35.2, U6.33 (PA12)
- no-connect marks 32 -> 38
Other:
- moved on the sheet: C1, C8, C9, D7, H1, H2, H3, H4, J1, J2, J3, J4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
